File: digitizer2.sch (KiCad schematic (older format))
At the start: 228 parts, among them P1 USB_OTG, P2 CONN_01X01, P3 CONN_01X01, P4 SMA, P5 SMA, P6 SMA, P7 CONN_02X03, P8 CONN_02X03, T1 ETC1-1-13, T2 ETC1-1-13, U1 XC7A35T, U10 SN65LVDS100DGK, U11 SN65LVDS100DGK, U12 ASTMLPA-18-100.000MHZ-EJ-E-T, U2 FT2232H, U3 MT41J128M16, U4 ADS5403, U5 LTC3569, U6 TPS79618DCQ, U7 TPS79633DCQ, U8 93LC46BT-I/OT, U9 LM3671MF-3.3, Y1 12MHz

Commit message: Start adding order codes
Parts:
- L3, L5, L6: OC_Farnell (none) -> 2056527
- L4: OC_Farnell (none) -> 2056528
- P4, P5, P6: OC_Farnell (none) -> 1248989
- T1, T2: OC_Digikey (none) -> 1465-1217-1-ND
- U1: OC_Digikey (none) -> 122-1912-ND
- U10, U11: OC_Farnell (none) -> 1607889
- U12: OC_Digikey (none) -> 535-13078-1-ND
- U2: value FT2232H -> FT2232HQ; OC_Digikey (none) -> 768-1025-1-ND
- U3: OC_Digikey (none) -> 557-1611-1-ND
- U4: OC_Digikey (none) -> 296-36911-5-ND
- U5: OC_Digikey (none) -> LTC3569EUD#PBF-ND
- U6: OC_Farnell (none) -> 2383027
- U7: OC_Farnell (none) -> 1207359
- U8: OC_Farnell (none) -> 1556164
- U9: OC_Farnell (none) -> 1685767
- Y1: OC_Farnell (none) -> 1841940
Changed lines of the file:
@@
 F 2 "SMD_Packages:BGA-256_pitch1mm_dia0.4mm" H 500 800 60  0001 C CNN
 F 3 "" H 500 800 60  0000 C CNN
+F 4 "122-1912-ND" H 500 800 60  0001 C CNN "OC_Digikey"
 	1    500  800
 	1    0    0    -1
@@
 P 3750 17100
 F 0 "U2" H 3750 17100 60  0000 C CNN
-F 1 "FT2232H" H 3750 17000 60  0000 C CNN
+F 1 "FT2232HQ" H 3750 17000 60  0000 C CNN
 F 2 "digitizer2_modules:QFN-FT2232HQ-64_pitch0.5" H 3750 17050 60  0001 C CNN
 F 3 "" H 3750 17050 60  0000 C CNN
+F 4 "768-1025-1-ND" H 3750 17100 60  0001 C CNN "OC_Digikey"
 	1    3750 17100
 	1    0    0    -1
@@
 F 2 "digitizer2_modules:BGA-196_pitch0.8mm_dia0.4mm" H 3400 31600 60  0001 C CNN
 F 3 "" H 3400 31600 60  0000 C CNN
+F 4 "296-36911-5-ND" H 3400 33450 60  0001 C CNN "OC_Digikey"
 	1    3400 33450
 	1    0    0    -1
@@
 F 2 "digitizer2_modules:BGA-96_pitch0.8mm_dia0.35mm" H 3500 22750 60  0001 C CNN
 F 3 "" H 3500 22750 60  0000 C CNN
+F 4 "557-1611-1-ND" H 3500 22800 60  0001 C CNN "OC_Digikey"
 	1    3500 22800
 	1    0    0    -1
@@
 F 2 "Housings_DFN_QFN:UQFN-20-1EP_3x3mm_Pitch0.4mm" H 2600 10300 60  0001 C CNN
 F 3 "" H 2600 10300 60  0000 C CNN
+F 4 "LTC3569EUD#PBF-ND" H 2600 10250 60  0001 C CNN "OC_Digikey"
 	1    2600 10250
 	1    0    0    -1
@@
 F 2 "digitizer2_modules:SOT-223-6" H 3400 29500 60  0001 C CNN
 F 3 "" H 3400 29500 60  0000 C CNN
+F 4 "2383027" H 3400 29500 60  0001 C CNN "OC_Farnell"
 	1    3400 29500
 	1    0    0    -1
@@
 F 2 "digitizer2_modules:SOT-223-6" H 3400 30550 60  0001 C CNN
 F 3 "" H 3400 30550 60  0000 C CNN
+F 4 "1207359" H 3400 30550 60  0001 C CNN "OC_Farnell"
 	1    3400 30550
 	1    0    0    -1
@@
 F 2 "digitizer2_modules:SOT-23-6" H 1150 18250 50  0001 C CNN
 F 3 "" H 1250 18350 50  0000 C CNN
+F 4 "1556164" H 1250 18250 60  0001 C CNN "OC_Farnell"
 	1    1250 18250
 	1    0    0    -1
@@
 F 2 "Crystals:Crystal_SMD_5032_2Pads" H 2350 18600 50  0001 C CNN
 F 3 "" H 2350 18600 50  0000 C CNN
+F 4 "1841940" H 2350 18600 60  0001 C CNN "OC_Farnell"
 	1    2350 18600
 	0    1    1    0
@@
 F 2 "TO_SOT_Packages_SMD:SOT-23-6" H 3100 12300 50  0001 C CNN
 F 3 "" H 3200 12400 50  0000 C CNN
+F 4 "1685767" H 3200 12300 60  0001 C CNN "OC_Farnell"
 	1    3200 12300
 	1    0    0    -1
@@
 F 2 "digitizer2_modules:IHLP-1212BZ-11" H 3850 12100 50  0001 C CNN
 F 3 "" H 3850 12100 50  0000 C CNN
+F 4 "2056527" V 3850 12100 60  0001 C CNN "OC_Farnell"
 	1    3850 12100
 	0    -1   -1   0
@@
 F 2 "digitizer2_modules:IHLP-1212BZ-11" H 3500 9550 50  0001 C CNN
 F 3 "" H 3500 9550 50  0000 C CNN
+F 4 "2056527" H 3500 9550 60  0001 C CNN "OC_Farnell"
 	1    3500 9550
 	1    0    0    -1
@@
 F 2 "digitizer2_modules:IHLP-1212BZ-11" H 3500 10250 50  0001 C CNN
 F 3 "" H 3500 10250 50  0000 C CNN
+F 4 "2056528" H 3500 10250 60  0001 C CNN "OC_Farnell"
 	1    3500 10250
 	1    0    0    -1
@@
 F 2 "digitizer2_modules:IHLP-1212BZ-11" H 3500 10950 50  0001 C CNN
 F 3 "" H 3500 10950 50  0000 C CNN
+F 4 "2056527" H 3500 10950 60  0001 C CNN "OC_Farnell"
 	1    3500 10950
 	1    0    0    -1
@@
 F 2 "Housings_SSOP:TSSOP-8_3x3mm_Pitch0.65mm" H 3650 26150 60  0001 C CNN
 F 3 "" H 3650 26150 60  0000 C CNN
+F 4 "1607889" H 3650 26150 60  0001 C CNN "OC_Farnell"
 	1    3650 26150
 	1    0    0    -1
@@
 F 2 "Housings_SSOP:TSSOP-8_3x3mm_Pitch0.65mm" H 3650 27250 60  0001 C CNN
 F 3 "" H 3650 27250 60  0000 C CNN
+F 4 "1607889" H 3650 27250 60  0001 C CNN "OC_Farnell"
 	1    3650 27250
 	1    0    0    -1
@@
 F 2 "digitizer2_modules:ETC1-1-13" V -1550 32450 50  0001 C CNN
 F 3 "" V -1550 32450 50  0000 C CNN
+F 4 "1465-1217-1-ND" H -1550 32450 60  0001 C CNN "OC_Digikey"
 	1    -1550 32450
 	1    0    0    1
@@
 F 2 "digitizer2_modules:ETC1-1-13" V -750 32450 50  0001 C CNN
 F 3 "" V -750 32450 50  0000 C CNN
+F 4 "1465-1217-1-ND" H -750 32450 60  0001 C CNN "OC_Digikey"
 	1    -750 32450
 	-1   0    0    -1
@@
 F 2 "digitizer2_modules:SMA_ANGLE_THT" H -3000 32250 50  0001 C CNN
 F 3 "" H -3000 32250 50  0000 C CNN
+F 4 "1248989" H -3000 32250 60  0001 C CNN "OC_Farnell"
 	1    -3000 32250
 	-1   0    0    -1
@@
 F 2 "digitizer2_modules:SMA_ANGLE_THT" H 1800 26100 50  0001 C CNN
 F 3 "" H 1800 26100 50  0000 C CNN
+F 4 "1248989" H 1800 26100 60  0001 C CNN "OC_Farnell"
 	1    1800 26100
 	-1   0    0    -1
@@
 F 2 "digitizer2_modules:SMA_ANGLE_THT" H 1800 27200 50  0001 C CNN
 F 3 "" H 1800 27200 50  0000 C CNN
+F 4 "1248989" H 1800 27200 60  0001 C CNN "OC_Farnell"
 	1    1800 27200
 	-1   0    0    -1
@@
 F 2 "digitizer2_modules:ASTMLPA" H -600 4100 60  0001 C CNN
 F 3 "" H -600 4100 60  0000 C CNN
+F 4 "535-13078-1-ND" H -600 4100 60  0001 C CNN "OC_Digikey"
 	1    -600 4100
 	1    0    0    -1

Commit message: Replace 47uF footprints with 0805. Rev 1.1
Parts:
- C129, C131, C142, C43, C49, C50, C52, C59, C66, C73: footprint Capacitors_SMD:C_0402 -> Capacitors_SMD:C_0805
Changed lines of the file:
@@
 F 0 "C43" H 3960 6970 50  0000 L CNN
 F 1 "47uF" H 3960 6820 50  0000 L CNN
-F 2 "Capacitors_SMD:C_0402" H 3950 6900 50  0001 C CNN
+F 2 "Capacitors_SMD:C_0805" H 3950 6900 50  0001 C CNN
 F 3 "" H 3950 6900 50  0000 C CNN
 	1    3950 6900
@@
 F 0 "C49" H 3960 7670 50  0000 L CNN
 F 1 "47uF" H 3960 7520 50  0000 L CNN
-F 2 "Capacitors_SMD:C_0402" H 3950 7600 50  0001 C CNN
+F 2 "Capacitors_SMD:C_0805" H 3950 7600 50  0001 C CNN
 F 3 "" H 3950 7600 50  0000 C CNN
 	1    3950 7600
@@
 F 0 "C50" H 4160 7670 50  0000 L CNN
 F 1 "47uF" H 4160 7520 50  0000 L CNN
-F 2 "Capacitors_SMD:C_0402" H 4150 7600 50  0001 C CNN
+F 2 "Capacitors_SMD:C_0805" H 4150 7600 50  0001 C CNN
 F 3 "" H 4150 7600 50  0000 C CNN
 	1    4150 7600
@@
 F 0 "C52" H 4710 7670 50  0000 L CNN
 F 1 "47uF" H 4710 7520 50  0000 L CNN
-F 2 "Capacitors_SMD:C_0402" H 4700 7600 50  0001 C CNN
+F 2 "Capacitors_SMD:C_0805" H 4700 7600 50  0001 C CNN
 F 3 "" H 4700 7600 50  0000 C CNN
 	1    4700 7600
@@
 F 0 "C59" H 4110 -30 50  0000 L CNN
 F 1 "47uF" H 4110 -180 50  0000 L CNN
-F 2 "Capacitors_SMD:C_0402" H 4100 -100 50  0001 C CNN
+F 2 "Capacitors_SMD:C_0805" H 4100 -100 50  0001 C CNN
 F 3 "" H 4100 -100 50  0000 C CNN
 	1    4100 -100
@@
 F 0 "C66" H 7010 20  50  0000 L CNN
 F 1 "47uF" H 7010 -130 50  0000 L CNN
-F 2 "Capacitors_SMD:C_0402" H 7000 -50 50  0001 C CNN
+F 2 "Capacitors_SMD:C_0805" H 7000 -50 50  0001 C CNN
 F 3 "" H 7000 -50 50  0000 C CNN
 	1    7000 -50
@@
 F 0 "C73" H 13460 120 50  0000 L CNN
 F 1 "47uF" H 13460 -30 50  0000 L CNN
-F 2 "Capacitors_SMD:C_0402" H 13450 50  50  0001 C CNN
+F 2 "Capacitors_SMD:C_0805" H 13450 50  50  0001 C CNN
 F 3 "" H 13450 50  50  0000 C CNN
 	1    13450 50
@@
 F 0 "C129" H 4175 28750 50  0000 L CNN
 F 1 "47uF" H 4175 28550 50  0000 L CNN
-F 2 "Capacitors_SMD:C_0402" H 4188 28500 50  0001 C CNN
+F 2 "Capacitors_SMD:C_0805" H 4188 28500 50  0001 C CNN
 F 3 "" H 4150 28650 50  0000 C CNN
 	1    4150 28650
@@
 F 0 "C131" H 525 16850 50  0000 L CNN
 F 1 "47uF" H 525 16650 50  0000 L CNN
-F 2 "Capacitors_SMD:C_0402" H 538 16600 50  0001 C CNN
+F 2 "Capacitors_SMD:C_0805" H 538 16600 50  0001 C CNN
 F 3 "" H 500 16750 50  0000 C CNN
 	1    500  16750
@@
 F 0 "C142" H 9610 20  50  0000 L CNN
 F 1 "47uF" H 9610 -130 50  0000 L CNN
-F 2 "Capacitors_SMD:C_0402" H 9600 -50 50  0001 C CNN
+F 2 "Capacitors_SMD:C_0805" H 9600 -50 50  0001 C CNN
 F 3 "" H 9600 -50 50  0000 C CNN
 	1    9600 -50

Commit message: Board revision 1.2
Parts:
- removed C10, C2, C21, C23, C24, C25, C26, C27, C28, C29, C30, C31, C32, C7: 4.7uF, Capacitors_SMD:C_0402, symbol C
- removed C143: 100nF, Capacitors_SMD:C_0402, symbol C
- removed JP3: JUMPER3, Pin_Headers:Pin_Header_Straight_1x03, symbol JUMPER3
- removed L3, L5: 2.2uH, digitizer2_modules:IHLP-1212BZ-11, symbol INDUCTOR_SMALL
- removed L4: 3.3uH, digitizer2_modules:IHLP-1212BZ-11, symbol INDUCTOR_SMALL
- removed L6: 2.2uH, digitizer2_modules:IHLP-1212BZ-11, symbol INDUCTOR
- removed R10: 175k, Resistors_SMD:R_0603, symbol R_Small
- removed R11, R15: 200k, Resistors_SMD:R_0603, symbol R_Small
- removed R12: 125k, Resistors_SMD:R_0603, symbol R_Small
- removed R13: 100k, Resistors_SMD:R_0603, symbol R_Small
- removed R14: 50k, Resistors_SMD:R_0603, symbol R_Small
- removed U12: ASTMLPA-18-100.000MHZ-EJ-E-T, digitizer2_modules:ASTMLPA, symbol OSCILLATOR_ABRACON
- removed U5: LTC3569, Housings_DFN_QFN:UQFN-20-1EP_3x3mm_Pitch0.4mm, symbol LTC3569
- removed Y1: 12MHz, Crystals:Crystal_SMD_5032_2Pads, symbol Crystal
- added C10, C149, C150, C151, C152, C153, C21, C23, C24, C25, C26, C27, C28, C29, C30, C31, C32, C7: 4.7uF, Capacitors_SMD:C_0402, symbol C_Small
- added C143, C159: 10nF, Capacitors_SMD:C_0402, symbol C_Small
- added C154, C160, C161, C162, C163, C164: 220uF, Capacitors_SMD:c_elec_5x5.7, symbol C_Small
- added C155, C156: 47uF, Capacitors_SMD:C_0805, symbol C_Small
- added C2: 100nF, Capacitors_SMD:C_0402, symbol C_Small
- added L15, L16, L3, L4, L5: ferrite, Resistors_SMD:R_0805, symbol INDUCTOR
- added L17, L18, L19, L20, L6: 2.2uH, digitizer2_modules:IHLP-1212BZ-11, symbol L_Small
- added R10: 4.7k, Resistors_SMD:R_0402, symbol R
- added R11: 0, Resistors_SMD:R_0603, symbol R
- added U12: ASG2-D-X-A-500.000MHZ, digitizer2_modules:ASG2, symbol OSCILLATOR_ASG2_D_X
- added U13: LM3671MF-1.8, TO_SOT_Packages_SMD:SOT-23-5, symbol LM3671
- added U14: LM3671MF-1.5, TO_SOT_Packages_SMD:SOT-23-5, symbol LM3671
- added U15: LM3671MF-2.5, TO_SOT_Packages_SMD:SOT-23-5, symbol LM3671
- added U16: FXO-LC526R-100, digitizer2_modules:FXO-LC52, symbol OSCILLATOR_FXO_LC52
- added U5: ADP2108AUJZ-1.0-R7, TO_SOT_Packages_SMD:SOT-23-5, symbol LM3671
- added Y1: ABM8G-12.000MHZ-18-D2Y-T, digitizer2_modules:ABM8G, symbol Crystal_ABM8G
- C18: value 20pF -> 100nF; footprint Capacitors_SMD:C_0603 -> Capacitors_SMD:C_0402
- C19, C20: value 20pF -> 4.7uF; footprint Capacitors_SMD:C_0603 -> Capacitors_SMD:C_0402
- P8: footprint Pin_Headers:Pin_Header_Angled_2x03 -> Pin_Headers:Pin_Header_Straight_2x03
- R6: value 200k -> 4.7k; footprint Resistors_SMD:R_0603 -> Resistors_SMD:R_0402
- U2: value FT2232HQ -> FT2232H-56Q; footprint digitizer2_modules:QFN-FT2232HQ-64_pitch0.5 -> digitizer2_modules:VQFN-FT2232H-56Q_pitch0.5; symbol FT2232H -> FT2232H-56Q
- U9: footprint TO_SOT_Packages_SMD:SOT-23-6 -> TO_SOT_Packages_SMD:SOT-23-5
Connections:
- net labels added: 1V0_REG, 1V5_REG, 1V8_REG, 2V5_REG, 3V3_REG, APWR_EN, GCLK_N, GCLK_P, USB_SIWUA, VDD_FPGA_2V5
- net labels removed: GCLK1
- wire segments 445 -> 533
- no-connect marks 98 -> 75
Other:
- note added: "VCC_AUX"
- note added: "VCC_CCO_DRAM"
- note added: "VCC_CCO_USB, VCC_FTDI"
- note added: "VCC_INT"
- note removed: "=1.76 MHz"
- note removed: "FB=0.8V"
- moved on the sheet: C122, C123, C124, C125, C126, C127, L7, L8, P7, U6, U7, U9

Commit message: New capacitor selection
Parts:
- removed C52: 47uF, Capacitors_SMD:C_0805, symbol C_Small
- removed L7, L8: ferrite, Resistors_SMD:R_0805, symbol INDUCTOR
- C1, C104, C105, C106, C107, C108, C109, C11, C116, C117, C118, C119, C12, C120, C121, C13, C132, C134, C14, C146, C148, C15, C16, C17, C18, C2, C22, C33, C34, C8, C80, C81, C82, C83, C84, C85, C92, C93, C94, C95, C96, C97: value 100nF -> 0.1uF
- C10, C122, C123, C125, C126, C128, C130, C140, C141, C149, C150, C151, C152, C153, C19, C20, C21, C23, C24, C25, C26, C27, C28, C29, C3, C30, C31, C32, C41, C42, C47, C48, C5, C57, C58, C64, C65, C7, C71, C72, C9: footprint Capacitors_SMD:C_0402 -> Capacitors_SMD:C_0805
- C129, C131, C142, C155, C156, C43, C49, C50, C59, C66, C73: footprint Capacitors_SMD:C_0805 -> Capacitors_SMD:C_1210
- C136, C137, C138, C139, C38, C39, C40, C44, C45, C46, C51, C53, C54, C55, C56, C60, C61, C62, C63, C67, C68, C69, C70: value 470nF -> 0.47uF
Connections:
- net A5V0: now also C125.1, U7.2 (IN)
- net VDD_ADC_3V3: now also C122.1, U6.2 (IN)

Commit message: Add 3.3V -> 2.5V regulator
Parts:
- removed C10, C149, C150, C151, C152, C153, C20, C21, C23, C24, C25, C26, C27, C28, C29, C30, C31, C32, C7: 4.7uF, Capacitors_SMD:C_0805, symbol C_Small
- removed C160, C161, C162, C163, C164: 220uF, Capacitors_SMD:c_elec_5x5.7, symbol C_Small
- removed L15, L16, L3, L4, L5: ferrite, Resistors_SMD:R_0805, symbol INDUCTOR
- removed L17, L18, L19, L20, L6: 2.2uH, digitizer2_modules:IHLP-1212BZ-11, symbol L_Small
- removed U13: LM3671MF-1.8, TO_SOT_Packages_SMD:SOT-23-5, symbol LM3671
- removed U14: LM3671MF-1.5, TO_SOT_Packages_SMD:SOT-23-5, symbol LM3671
- removed U15: LM3671MF-2.5, TO_SOT_Packages_SMD:SOT-23-5, symbol LM3671
- removed U5: ADP2108AUJZ-1.0-R7, TO_SOT_Packages_SMD:SOT-23-5, symbol LM3671
- removed U9: LM3671MF-3.3, TO_SOT_Packages_SMD:SOT-23-5, symbol LM3671MF-3.3
- added C10, C7: 4.7uF, Capacitors_SMD:C_0805, symbol C
- added JP3: JUMPER, Pin_Headers:Pin_Header_Straight_1x02, symbol JUMPER
- added U5: TPS79625DCQ, digitizer2_modules:SOT-223-6, symbol TPS79618DCQ
- C19: value 4.7uF -> 10nF; footprint Capacitors_SMD:C_0805 -> Capacitors_SMD:C_0402
Connections:
- net 5V0: no longer C19.1
- net GND: now also C10.2, C7.2, U5.3 (GND), U5.6 (PAD)
- net VDD_FPGA_2V5: now also C10.1, U5.4 (OUT)
- net VDD_FPGA_3V3: now also JP3.1
- new net: C7.1, JP3.2, U5.1 (EN), U5.2 (IN)
- new net: C19.1, U5.5 (NR)
Other:
- note removed: "VCC_AUX"
- note removed: "VCC_CCO_DRAM"
- note removed: "VCC_CCO_USB, VCC_FTDI"
- note removed: "VCC_INT"
